File: stepper_tmc_max22210.kicad_sch (KiCad schematic)
At the start: 13 parts, among them J1 Conn_01x08_pin, J2 Conn_01x08_pin, M1 Stepper_Motor_bipolar, U1 MAX22210ATJ+

Commit message: Finished functional design, ready for silk screen and BOM revision
Connections:
- net RESET is gone; now on net SLEEP: J1.4 (Pin_4)
- net VDD is gone; now on net +1V8: J2.7 (Pin_7)
- net VMOT is gone; now on net +VDC: J2.1 (Pin_1)
- net M1: now also U1.20 (OUT2B); no longer U1.21 (OUT2A)
- net M2: now also U1.18 (OUT1B); no longer U1.23 (OUT1A)
- net M3: now also U1.21 (OUT2A); no longer U1.20 (OUT2B)
- net M4: now also U1.23 (OUT1A); no longer U1.18 (OUT1B)
Changed lines of the file:
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@@
 	)
 	(junction
+		(at 72.39 50.8)
+		(diameter 0)
+		(color 0 0 0 0)
+	)
+	(junction
 		(at 157.48 39.37)
 		(diameter 0)
@@
 	(wire
 		(pts
-			(xy 172.72 64.77) (xy 173.99 64.77)
+			(xy 232.41 73.66) (xy 233.68 73.66)
 		)
 		(stroke
@@
 	(wire
 		(pts
-			(xy 232.41 73.66) (xy 233.68 73.66)
+			(xy 96.52 44.45) (xy 109.22 44.45)
 		)
 		(stroke
@@
 	(wire
 		(pts
-			(xy 96.52 44.45) (xy 109.22 44.45)
+			(xy 91.44 72.39) (xy 88.9 74.93)
 		)
 		(stroke
@@
 	(wire
 		(pts
-			(xy 91.44 72.39) (xy 88.9 74.93)
+			(xy 163.83 46.99) (xy 165.1 45.72)
 		)
 		(stroke
@@
 	(wire
 		(pts
-			(xy 163.83 46.99) (xy 165.1 45.72)
+			(xy 224.79 43.18) (xy 224.79 44.45)
 		)
 		(stroke
@@
 	(wire
 		(pts
-			(xy 224.79 43.18) (xy 224.79 44.45)
+			(xy 64.77 50.8) (xy 72.39 50.8)
 		)
 		(stroke
@@
 	(wire
 		(pts
+			(xy 173.99 64.77) (xy 172.72 64.77)
+		)
+		(stroke
+			(width 0)
+			(type default)
+		)
+	)
+	(wire
+		(pts
 			(xy 173.99 64.77) (xy 182.88 64.77)
 		)
@@
 		)
 	)
+	(wire
+		(pts
+			(xy 72.39 50.8) (xy 72.39 52.07)
+		)
+		(stroke
+			(width 0)
+			(type default)
+		)
+	)
 	(polyline
 		(pts
@@
 	(wire
 		(pts
-			(xy 72.39 48.26) (xy 72.39 52.07)
+			(xy 72.39 48.26) (xy 72.39 50.8)
 		)
 		(stroke
@@
 		)
 	)
+	(global_label "VDD"
+		(shape input)
+		(at 64.77 50.8 180)
+		(fields_autoplaced yes)
+		(effects
+			(font
+				(face "Monospac821 BT")
+				(size 1.27 1.27)
+			)
+			(justify right)
+		)
+		(property "Intersheetrefs" "${INTERSHEET_REFS}"
+			(at 58.7987 50.8 0)
+			(effects
+				(font
+					(size 1.27 1.27)
+				)
+				(justify right)
+				(hide yes)
+			)
+		)
+	)
 	(global_label "M3"
 		(shape input)
@@
 	(global_label "M1"
 		(shape input)
-		(at 156.21 67.31 0)
+		(at 156.21 69.85 0)
 		(fields_autoplaced yes)
 		(effects
@@
 		)
 		(property "Intersheetrefs" "${INTERSHEET_REFS}"
-			(at 161.8561 67.31 0)
+			(at 161.8561 69.85 0)
 			(effects
 				(font
@@
 	(global_label "M2"
 		(shape input)
-		(at 156.21 62.23 0)
+		(at 156.21 74.93 0)
 		(fields_autoplaced yes)
 		(effects
@@
 		)
 		(property "Intersheetrefs" "${INTERSHEET_REFS}"
-			(at 161.8561 62.23 0)
+			(at 161.8561 74.93 0)
 			(effects
 				(font
@@
 		)
 	)
-	(global_label "STEP"
+	(global_label "SLEEP"
 		(shape input)
-		(at 106.68 54.61 180)
+		(at 210.82 71.12 0)
 		(fields_autoplaced yes)
 		(effects
 			(font
+				(face "Monospac821 BT")
 				(size 1.27 1.27)
 			)
-			(justify right)
+			(justify left)
 		)
 		(property "Intersheetrefs" "${INTERSHEET_REFS}"
-			(at 99.0987 54.61 0)
+			(at 218.9304 71.12 0)
 			(effects
 				(font
 					(size 1.27 1.27)
 				)
-				(justify right)
+				(justify left)
 				(hide yes)
 			)
 		)
 	)
-	(global_label "M3"
+	(global_label "STEP"
 		(shape input)
-		(at 156.21 69.85 0)
+		(at 106.68 54.61 180)
 		(fields_autoplaced yes)
 		(effects
@@
 				(size 1.27 1.27)
 			)
-			(justify left)
+			(justify right)
 		)
 		(property "Intersheetrefs" "${INTERSHEET_REFS}"
-			(at 161.8561 69.85 0)
+			(at 99.0987 54.61 0)
 			(effects
 				(font
 					(size 1.27 1.27)
 				)
-				(justify left)
+				(justify right)
 				(hide yes)
 			)
 		)
 	)
-	(global_label "hfs_select"
+	(global_label "M3"
 		(shape input)
-		(at 88.9 57.15 180)
+		(at 156.21 67.31 0)
 		(fields_autoplaced yes)
 		(effects
@@
 				(size 1.27 1.27)
 			)
-			(justify right)
+			(justify left)
 		)
 		(property "Intersheetrefs" "${INTERSHEET_REFS}"
-			(at 76.3596 57.15 0)
+			(at 161.8561 67.31 0)
 			(effects
 				(font
 					(size 1.27 1.27)
 				)
-				(justify right)
+				(justify left)
 				(hide yes)
 			)
 		)
 	)
-	(global_label "RESET"
+	(global_label "hfs_select"
 		(shape input)
-		(at 210.82 71.12 0)
+		(at 88.9 57.15 180)
 		(fields_autoplaced yes)
 		(effects
 			(font
-				(face "Monospac821 BT")
 				(size 1.27 1.27)
 			)
-			(justify left)
+			(justify right)
 		)
 		(property "Intersheetrefs" "${INTERSHEET_REFS}"
-			(at 218.9304 71.12 0)
+			(at 76.3596 57.15 0)
 			(effects
 				(font
 					(size 1.27 1.27)
 				)
-				(justify left)
+				(justify right)
 				(hide yes)
 			)
@@
 	(global_label "M4"
 		(shape input)
-		(at 156.21 74.93 0)
+		(at 156.21 62.23 0)
 		(fields_autoplaced yes)
 		(effects
@@
 		)
 		(property "Intersheetrefs" "${INTERSHEET_REFS}"
-			(at 161.8561 74.93 0)
+			(at 161.8561 62.23 0)
 			(effects
 				(font
@@
 				(hide yes)
 			)
+		)
+	)
+	(global_label "VMOT"
+		(shape input)
+		(at 173.99 62.23 180)
+		(fields_autoplaced yes)
+		(effects
+			(font
+				(face "Monospac821 BT")
+				(size 1.27 1.27)
+			)
+			(justify right)
+		)
+		(property "Intersheetrefs" "${INTERSHEET_REFS}"
+			(at 166.9491 62.23 0)
+			(effects
+				(font
+					(size 1.27 1.27)
+				)
+				(justify right)
+				(hide yes)
+			)
